File: EAGLE_BOT/PAGE1.brd (EAGLE design)
At the start: 160 x 160 mm, 101 parts, among them Q1 IRF640, U1 NE555_SOP8, U10 NE556_SOP14, U11 4017_SOP16, U12 4017_SOP16, U13 4518_SMD, U14 4510_DIP, U15 4001_SOP14, U16 4081, U2 4040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

Commit message: ver1 Complete
Parts:
- removed R47: 20K, !JKS:SMD2012
- added C10: 100uF, !JKS:CAP_POL_BIG
- added R17, R22, R23: 47k, !JKS:SMD2012
Connections:
- net +5V: now also C10.1; no longer R47.1
- net FASTER_CV: no longer R47.2
- net GND: now also C10.2, R17.2, R22.2, R23.2
- net LED_CON_1: now also R17.1
- net LED_CON_2: now also R22.1
- net LED_CON_3: now also R23.1
Routing:
- net N$60: track 264.4 -> 267.8 mm
- net N$6: track 201.9 -> 205.0 mm
- net MOD_FASTER: track 318.5 -> 321.5 mm
- net LED_CON_G: track 198.2 -> 201.2 mm
- net FASTER_CV: track 85.0 -> 88.0 mm
- net MOD_FAST3: track 303.3 -> 305.9 mm
- net LED_CON_2: track 189.4 -> 192.1 mm
- net MOD_SW: track 189.7 -> 192.2 mm
- net LED_CON_B: track 211.8 -> 214.2 mm
- net LED_CON_1: track 188.5 -> 190.3 mm
- net N$77: track 233.8 -> 235.6 mm
- net N$9: track 88.3 -> 89.9 mm
- net N$26: track 114.8 -> 116.5 mm
- net N$63: track 77.7 -> 76.4 mm
- net N$5: track 44.5 -> 43.3 mm
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Other:
- board text added: "Designed by JsKim"
- board text removed: "TREE_BOTTOM"
