File: EAGLE_BOT/PAGE1.sch (EAGLE design)
At the start: 101 parts, among them Q1 IRF640, U1 NE555_SOP8, U10 NE556_SOP14, U11 4017_SOP16, U12 4017_SOP16, U13 4518_SMD, U14 4510_DIP, U15 4001_SOP14, U16 4081, U2 4040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

Commit message: ver1 Complete
Parts:
- removed R47: 20K, !JKS:RES_2012
- added C10: 100uF, !JKS:CAP_POL_BIG
- added R17, R22, R23: 47k, !JKS:RES_2012
Connections:
- net +5V: now also C10.1; no longer R47.1
- net FASTER_CV: no longer R47.2
- net GND: now also C10.2, R17.2, R22.2, R23.2
- net LED_CON_1: now also R17.1
- net LED_CON_2: now also R22.1
- net LED_CON_3: now also R23.1
Other:
- moved on the sheet: P1
Changed lines of the file:
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@@
 </variantdefs>
 <classes>
-<class number="0" name="default" width="0.254" drill="0.8">
+<class number="0" name="default" width="0.254" drill="0">
 </class>
-<class number="1" name="POWER" width="0.3" drill="0.8">
+<class number="1" name="POWER" width="0.3" drill="0">
 </class>
 </classes>
@@
 <part name="R46" library="!JKS" deviceset="RES" device="_2012" value="20K"/>
 <part name="GND37" library="!JKS" deviceset="GND" device=""/>
-<part name="R47" library="!JKS" deviceset="RES" device="_2012" value="20K"/>
-<part name="+5V27" library="!JKS" deviceset="+5V" device=""/>
 <part name="R48" library="!JKS" deviceset="RES" device="_2012" value="10K"/>
 <part name="C20" library="!JKS" deviceset="CAP_NP" device="_SMD2012" value="0.1uF"/>
@@
 <part name="NC35" library="!JKS" deviceset="NC" device=""/>
 <part name="NC36" library="!JKS" deviceset="NC" device=""/>
+<part name="R17" library="!JKS" deviceset="RES" device="_2012" value="47k"/>
+<part name="R22" library="!JKS" deviceset="RES" device="_2012" value="47k"/>
+<part name="R23" library="!JKS" deviceset="RES" device="_2012" value="47k"/>
+<part name="GND14" library="!JKS" deviceset="GND" device=""/>
+<part name="GND15" library="!JKS" deviceset="GND" device=""/>
+<part name="GND42" library="!JKS" deviceset="GND" device=""/>
+<part name="C10" library="!JKS" deviceset="CAP_POL" device="_BIG" value="100uF"/>
 </parts>
 <sheets>
@@
 <attribute name="VALUE" x="353.06" y="110.236" size="1.778" layer="96" align="center"/>
 </instance>
-<instance part="R47" gate="G$1" x="327.66" y="48.26" smashed="yes" rot="R90">
-<attribute name="NAME" x="325.12" y="50.8" size="1.778" layer="95"/>
-<attribute name="VALUE" x="324.612" y="43.688" size="1.778" layer="96"/>
-</instance>
-<instance part="+5V27" gate="G$1" x="304.8" y="63.5" smashed="yes">
-<attribute name="VALUE" x="304.8" y="67.31" size="1.27" layer="96" align="center"/>
-</instance>
 <instance part="R48" gate="G$1" x="157.48" y="27.94" smashed="yes">
 <attribute name="NAME" x="158.75" y="27.94" size="1.778" layer="95"/>
@@
 <attribute name="VALUE" x="259.08" y="209.296" size="1.778" layer="96" align="center"/>
 </instance>
-<instance part="P1" gate="G$1" x="342.9" y="195.58" smashed="yes">
-<attribute name="NAME" x="337.566" y="201.422" size="1.778" layer="95"/>
-</instance>
-<instance part="+5V30" gate="G$1" x="358.14" y="205.74" smashed="yes">
-<attribute name="VALUE" x="358.14" y="209.55" size="1.27" layer="96" align="center"/>
-</instance>
-<instance part="GND40" gate="G$1" x="358.14" y="185.42" smashed="yes">
-<attribute name="VALUE" x="358.14" y="181.356" size="1.778" layer="96" align="center"/>
+<instance part="P1" gate="G$1" x="43.18" y="236.22" smashed="yes">
+<attribute name="NAME" x="37.846" y="242.062" size="1.778" layer="95"/>
+</instance>
+<instance part="+5V30" gate="G$1" x="58.42" y="246.38" smashed="yes">
+<attribute name="VALUE" x="58.42" y="250.19" size="1.27" layer="96" align="center"/>
+</instance>
+<instance part="GND40" gate="G$1" x="58.42" y="226.06" smashed="yes">
+<attribute name="VALUE" x="58.42" y="221.996" size="1.778" layer="96" align="center"/>
+</instance>
+<instance part="R17" gate="G$1" x="302.26" y="165.1" smashed="yes">
+<attribute name="NAME" x="303.53" y="165.1" size="1.778" layer="95"/>
+<attribute name="VALUE" x="303.53" y="162.56" size="1.778" layer="96"/>
+</instance>
+<instance part="R22" gate="G$1" x="309.88" y="165.1" smashed="yes">
+<attribute name="NAME" x="311.15" y="165.1" size="1.778" layer="95"/>
+<attribute name="VALUE" x="311.15" y="162.56" size="1.778" layer="96"/>
+</instance>
+<instance part="R23" gate="G$1" x="317.5" y="165.1" smashed="yes">
+<attribute name="NAME" x="318.77" y="165.1" size="1.778" layer="95"/>
+<attribute name="VALUE" x="318.77" y="162.56" size="1.778" layer="96"/>
+</instance>
+<instance part="GND14" gate="G$1" x="302.26" y="157.48" smashed="yes">
+<attribute name="VALUE" x="302.26" y="153.416" size="1.778" layer="96" align="center"/>
+</instance>
+<instance part="GND15" gate="G$1" x="309.88" y="157.48" smashed="yes">
+<attribute name="VALUE" x="309.88" y="153.416" size="1.778" layer="96" align="center"/>
+</instance>
+<instance part="GND42" gate="G$1" x="317.5" y="157.48" smashed="yes">
+<attribute name="VALUE" x="317.5" y="153.416" size="1.778" layer="96" align="center"/>
+</instance>
+<instance part="C10" gate="G$1" x="66.04" y="238.76" smashed="yes">
+<attribute name="NAME" x="71.12" y="238.76" size="1.27" layer="95"/>
+<attribute name="VALUE" x="71.12" y="236.982" size="1.27" layer="95"/>
 </instance>
 </instances>
@@
 <pinref part="P1" gate="G$1" pin="-"/>
 <pinref part="GND40" gate="G$1" pin="GND"/>
-<wire x1="353.06" y1="193.04" x2="358.14" y2="193.04" width="0.1524" layer="91"/>
-<wire x1="358.14" y1="193.04" x2="358.14" y2="187.96" width="0.1524" layer="91"/>
+<wire x1="53.34" y1="233.68" x2="58.42" y2="233.68" width="0.1524" layer="91"/>
+<wire x1="58.42" y1="233.68" x2="58.42" y2="231.14" width="0.1524" layer="91"/>
+<pinref part="C10" gate="G$1" pin="2"/>
+<wire x1="58.42" y1="231.14" x2="58.42" y2="228.6" width="0.1524" layer="91"/>
+<wire x1="66.04" y1="233.68" x2="66.04" y2="231.14" width="0.1524" layer="91"/>
+<wire x1="66.04" y1="231.14" x2="58.42" y2="231.14" width="0.1524" layer="91"/>
+<junction x="58.42" y="231.14"/>
+</segment>
+<segment>
+<pinref part="R17" gate="G$1" pin="2"/>
+<pinref part="GND14" gate="G$1" pin="GND"/>
+</segment>
+<segment>
+<pinref part="R22" gate="G$1" pin="2"/>
+<pinref part="GND15" gate="G$1" pin="GND"/>
+</segment>
+<segment>
+<pinref part="R23" gate="G$1" pin="2"/>
+<pinref part="GND42" gate="G$1" pin="GND"/>
 </segment>
 </net>
@@
 </segment>
 <segment>
-<pinref part="+5V27" gate="G$1" pin="+5V"/>
-<pinref part="R47" gate="G$1" pin="1"/>
-<wire x1="304.8" y1="60.96" x2="304.8" y2="48.26" width="0.1524" layer="91"/>
-<wire x1="304.8" y1="48.26" x2="322.58" y2="48.26" width="0.1524" layer="91"/>
-</segment>
-<segment>
 <pinref part="+5V28" gate="G$1" pin="+5V"/>
 <pinref part="C26" gate="G$1" pin="1"/>
@@
 <pinref part="P1" gate="G$1" pin="+"/>
 <pinref part="+5V30" gate="G$1" pin="+5V"/>
-<wire x1="353.06" y1="198.12" x2="358.14" y2="198.12" width="0.1524" layer="91"/>
-<wire x1="358.14" y1="198.12" x2="358.14" y2="203.2" width="0.1524" layer="91"/>
+<wire x1="53.34" y1="238.76" x2="58.42" y2="238.76" width="0.1524" layer="91"/>
+<wire x1="58.42" y1="238.76" x2="58.42" y2="241.3" width="0.1524" layer="91"/>
+<pinref part="C10" gate="G$1" pin="1"/>
+<wire x1="58.42" y1="241.3" x2="58.42" y2="243.84" width="0.1524" layer="91"/>
+<wire x1="58.42" y1="241.3" x2="66.04" y2="241.3" width="0.1524" layer="91"/>
+<junction x="58.42" y="241.3"/>
 </segment>
 </net>
@@
 <segment>
 <pinref part="D9" gate="G$1" pin="2"/>
-<wire x1="299.72" y1="215.9" x2="320.04" y2="215.9" width="0.1524" layer="91"/>
-<label x="304.8" y="215.9" size="1.778" layer="95"/>
+<wire x1="299.72" y1="215.9" x2="302.26" y2="215.9" width="0.1524" layer="91"/>
+<label x="322.58" y="215.9" size="1.778" layer="95"/>
+<pinref part="R17" gate="G$1" pin="1"/>
+<wire x1="302.26" y1="215.9" x2="337.82" y2="215.9" width="0.1524" layer="91"/>
+<wire x1="302.26" y1="170.18" x2="302.26" y2="215.9" width="0.1524" layer="91"/>
+<junction x="302.26" y="215.9"/>
 </segment>
 <segment>
@@
 </segment>
 <segment>
-<wire x1="299.72" y1="195.58" x2="320.04" y2="195.58" width="0.1524" layer="91"/>
+<wire x1="299.72" y1="195.58" x2="309.88" y2="195.58" width="0.1524" layer="91"/>
 <pinref part="D10" gate="G$1" pin="2"/>
-<label x="304.8" y="195.58" size="1.778" layer="95"/>
+<label x="322.58" y="195.58" size="1.778" layer="95"/>
+<pinref part="R22" gate="G$1" pin="1"/>
+<wire x1="309.88" y1="195.58" x2="337.82" y2="195.58" width="0.1524" layer="91"/>
+<wire x1="309.88" y1="170.18" x2="309.88" y2="195.58" width="0.1524" layer="91"/>
+<junction x="309.88" y="195.58"/>
 </segment>
 <segment>
@@
 </segment>
 <segment>
-<wire x1="299.72" y1="175.26" x2="320.04" y2="175.26" width="0.1524" layer="91"/>
+<wire x1="299.72" y1="175.26" x2="317.5" y2="175.26" width="0.1524" layer="91"/>
 <pinref part="D11" gate="G$1" pin="2"/>
-<label x="304.8" y="175.26" size="1.778" layer="95"/>
+<label x="322.58" y="175.26" size="1.778" layer="95"/>
+<pinref part="R23" gate="G$1" pin="1"/>
+<wire x1="317.5" y1="175.26" x2="337.82" y2="175.26" width="0.1524" layer="91"/>
+<wire x1="317.5" y1="170.18" x2="317.5" y2="175.26" width="0.1524" layer="91"/>
+<junction x="317.5" y="175.26"/>
 </segment>
 <segment>
@@
 <pinref part="R45" gate="G$1" pin="2"/>
 <wire x1="332.74" y1="60.96" x2="335.28" y2="60.96" width="0.1524" layer="91"/>
-<pinref part="R47" gate="G$1" pin="2"/>
-<wire x1="332.74" y1="48.26" x2="335.28" y2="48.26" width="0.1524" layer="91"/>
-<wire x1="335.28" y1="48.26" x2="335.28" y2="60.96" width="0.1524" layer="91"/>
 <junction x="335.28" y="60.96"/>
 <wire x1="335.28" y1="60.96" x2="353.06" y2="60.96" width="0.1524" layer="91"/>
