File: Tree1/tree1.brd (EAGLE design)
At the start: 115 x 145 mm, 25 parts, among them CON1 TREE_CON_SINGLE, CON2 SOLDER_CON_2, CON3 SOLDER_CON_2

Commit message: ver1 Complete
Parts:
- moved CON3 7.33 mm to (39.8, 54.9)
- moved CON2 3.53 mm to (39.8, 67.0)
- moved R3 0.38 mm to (30.4, 70.0)
Routing:
- net LED_ARR3: track 151.2 -> 164.3 mm
- net LED_ARR1: track 128.7 -> 134.4 mm
- net LED_ARR2: track 167.9 -> 172.1 mm
- net +5V: track 298.5 -> 301.7 mm
