File: Tree2/tree2.brd (EAGLE design)
At the start: 115 x 145 mm, 25 parts, among them CON1 TREE_CON_SINGLE, CON2 SOLDER_CON_2, CON3 SOLDER_CON_2

Commit message: Operation Complete
Changed lines of the file:
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@@
 <contactref element="B" pad="1"/>
 <contactref element="CON1" pad="2"/>
-<wire x1="47.08" y1="139.15" x2="45.7" y2="137.77" width="0.254" layer="16"/>
 <wire x1="45.7" y1="73.7" x2="46.6" y2="72.8" width="0.254" layer="16"/>
 <via x="46.6" y="72.8" extent="1-16" drill="0.8" diameter="1.6"/>
@@
 <wire x1="46.5" y1="55.8" x2="46.6" y2="55.7" width="0.254" layer="1"/>
 <via x="46.6" y="55.7" extent="1-16" drill="0.8" diameter="1.6"/>
-<wire x1="45.7" y1="137.77" x2="45.7" y2="73.7" width="0.254" layer="16"/>
+<wire x1="45.7" y1="131.9" x2="45.7" y2="73.7" width="0.254" layer="16"/>
 <wire x1="46.6" y1="55.7" x2="46.6" y2="50.3" width="0.254" layer="16"/>
 <wire x1="62.453" y1="34.447" x2="62.453" y2="3.621" width="0.254" layer="16"/>
 <wire x1="46.6" y1="50.3" x2="62.453" y2="34.447" width="0.254" layer="16"/>
+<wire x1="47.08" y1="139.15" x2="47.08" y2="133.28" width="0.254" layer="16"/>
+<wire x1="47.08" y1="133.28" x2="45.7" y2="131.9" width="0.254" layer="16"/>
 </signal>
 </signals>

Commit message: ver1 Complete
Parts:
- moved CON3 9.56 mm to (45.3, 51.3)
- moved CON2 6.07 mm to (45.2, 63.0)
Routing:
- net +5V: track 369.5 -> 374.6 mm
- net LED_ARR3: track 257.8 -> 254.2 mm
- net LED_ARR2: track 257.6 -> 258.8 mm
- net RGB_B: track 143.1 -> 144.1 mm
Other:
- outline, holes or cut-outs redrawn
